File: Hardware/STAUB_BLIZZARD_107L/MowerBoard.kicad_pcb (KiCad board)
At the start: 4 copper layers, 54 x 120 mm, 99 parts, among them IC1 TPS62162DSGR, IC2 MC33978AES, IC3 PTPS274C65ASRHAR, IC4 TPS7B8601QDDARQ1, J1 432550083, J2 43045-0227, J3 39-28-1143, J4 SMA-J-P-H-ST-TH1, K1 V23086C2001A403, K2 V23086C2001A403, U1 AVR128DB48x-x6LX, U2 317990687

Commit message: RC2 du PCB, corrigé taille des vias et isolation. Ajout via GND. Reprise des leds de status
Parts:
- C29: moved to F.Cu
- IC2: footprint SamacSys_Parts:QFN50P500X500X90-33N-D -> Custom:QFN50P500X500X90-33N-D_Pasta
- IC3: footprint SamacSys_Parts:QFN50P600X600X100-41N-D -> Custom:QFN50P600X600X100-41N-D_pasta
- moved C29 2.45 mm to (126.8, 55.5), turned to 180 degrees
- turned D11 to 0 degrees
- turned D12 to 0 degrees
- turned D14 to 0 degrees
- turned D9 to 0 degrees
Routing:
- net Net-(D12-K): track 13.3 -> 7.25 mm
- net Net-(D10-A): track 15.8 -> 10.2 mm
- net /OUT/LEDOUT3: track 39.6 -> 37.6 mm, vias 3 -> 2
- net Net-(IC2-SP4): track 33.3 -> 35.1 mm
- net Net-(IC2-SP5): track 30.8 -> 32.3 mm
- net MISO: track 76.3 -> 77.6 mm
- net GND: track 28.8 -> 28.1 mm, vias 106 -> 163
- net INT_IC2: track 13.3 -> 14.0 mm
- net AMUX_IC2: track 13.5 -> 14.2 mm
- net Net-(IC2-SP6): track 29.5 -> 30.2 mm
- net /MCU/UPDI: vias 0 -> 1
- net +BATT: vias 7 -> 8
- net (no net): vias 6 -> 0

Commit message: Travail sur le BOM, changement de quelques empreintes pour aligner sur les disponibilités
Parts:
- added C34: 2.2uF 15V, Capacitor_SMD:C_0603_1608Metric, F.Cu at (127.8, 101.7)
- added C35: 100nF 15V, Capacitor_SMD:C_0402_1005Metric, F.Cu at (124.4, 97.4)
- C1: value 1uF -> 1uF 15V
- C10: value 1uF -> 10uF 50V; footprint Capacitor_SMD:C_0805_2012Metric -> Capacitor_SMD:C_1206_3216Metric
- C11, C13, C33, C4, C5: value 4.7 µF -> 4.7uF 15V; footprint Capacitor_SMD:C_0402_1005Metric -> Capacitor_SMD:C_0603_1608Metric
- C12, C14, C3: value 100 nF -> 100nF 15V
- C15, C16, C17, C18, C19, C2, C22, C23, C24, C25, C27: value 0.1uF -> 100nF 50V; footprint Capacitor_SMD:C_0402_1005Metric -> Capacitor_SMD:C_0603_1608Metric
- C26: value 100uF -> 100uF 50V; footprint Capacitor_SMD:CP_Elec_6.3x5.7 -> Capacitor_SMD:CP_Elec_8x10
- C28: value 1nF -> 1nF 50V
- C29: value 0.1uF -> 100nF 15V
- C30: value 100pF -> 100pF 15V
- C31: value 4.7nF -> 4.7nF 50V
- C32: value 100nF -> 100nF 50V
- C6: value 10uF -> 10uF 25V
- C7: value 22uF -> 22uF 16V
- C8: value 100uF -> 100uF Polym 10v
- C9: value 10uF -> 10uF 50V; footprint Capacitor_SMD:C_0805_2012Metric -> Capacitor_SMD:C_1206_3216Metric
- D16, D17, D8: value D_Schottky_Small -> PMEG60T30ELR-QX
- FB1: value FerriteBead_Small -> ILHB0603ER601VHC41
- IC4: footprint SamacSys_Parts:SOIC127P600X170-9N -> Custom:SOIC127P600X170-9N_pasta
- R10, R11, R14, R15, R16, R17, R6, R7, R8, R9: value 100 -> 100 1/4W
- R23: value 1k -> 33k 1/4W
- R24: value 1k -> 100k
- R28: value 22 -> 470
- R4, R5: value R_Small -> 390
- TP3: value +5V -> +3.3v
- U1: footprint Package_DFN_QFN:QFN-48-1EP_6x6mm_P0.4mm_EP4.2x4.2mm -> Package_DFN_QFN:VQFN-48-1EP_6x6mm_P0.4mm_EP4.1x4.1mm
- moved C19 4.73 mm to (120.9, 69.2)
- moved R11 4.49 mm to (119.4, 69.2)
- moved C18 4.24 mm to (117.8, 69.2)
- moved D19 4.15 mm to (107.8, 104.5), turned to 90 degrees
- moved R10 3.99 mm to (116.2, 69.2)
- moved C22 3.74 mm to (114.7, 69.2)
- moved R14 3.50 mm to (113.1, 69.2)
- moved C23 3.24 mm to (111.6, 69.2)
- moved C26 3.05 mm to (98.0, 103.6), turned to -90 degrees
- moved R15 3.00 mm to (110.0, 69.2)
- moved C24 2.75 mm to (108.5, 69.2)
- moved R16 2.51 mm to (106.9, 69.2)
- moved C25 2.25 mm to (105.4, 69.2)
- moved R17 2.02 mm to (103.8, 69.2)
- moved C17 1.76 mm to (102.2, 69.2)
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Connections:
- C26 pad 1: GND -> +BATT
- C26 pad 2: +BATT -> GND
Routing:
- net VCC: track 29.9 -> 34.6 mm
- net /INPUT_START: track 14.6 -> 10.9 mm
- net /INPUT_SEAT: track 10.1 -> 13.5 mm
- net Net-(IC2-SG0): track 13.8 -> 11.0 mm
- net Net-(IC2-SP7): track 26.3 -> 23.6 mm
- net Net-(IC2-SP6): track 30.2 -> 27.9 mm
- net Net-(IC2-SG1): track 11.4 -> 9.21 mm
- net /INPUT_BRAKE: track 9.44 -> 11.5 mm
- net GND: track 28.1 -> 26.1 mm, vias 163 -> 154
- net Net-(IC2-SP0): track 35.5 -> 37.3 mm
- net Net-(IC2-SP4): track 35.1 -> 33.5 mm
- net Net-(IC2-SP5): track 32.3 -> 30.7 mm
- net /INPUT_PTO_GS: track 15.2 -> 16.3 mm
- net Net-(IC2-SP3): track 27.0 -> 26.1 mm
- net /INPUT_FORWARD: track 9.90 -> 10.7 mm
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
Commit message: Ajout du connecteur de programmation du module Lora
Parts:
- removed the D17 at (121.3, 31.8)
- removed the D5 at (115.5, 104.3)
- added D19: 1N4148W, Diode_SMD:D_SOD-123, F.Cu at (115.5, 104.3)
- added D6: BAT54W, Package_TO_SOT_SMD:SOT-323_SC-70, F.Cu at (80.0, 43.8)
- added D7: BAT54W, Package_TO_SOT_SMD:SOT-323_SC-70, F.Cu at (122.7, 32.0)
- added SW1: ~, Connector_PinHeader_2.54mm:PinHeader_1x04_P2.54mm_Vertical, F.Cu at (92.8, 50.0)
- added UART1: ~, Connector_PinHeader_2.54mm:PinHeader_1x04_P2.54mm_Vertical, F.Cu at (80.0, 40.2)
- moved C7 0.65 mm to (119.5, 40.5)
- moved C6 0.57 mm to (119.1, 39.2)
- renumbered C30 to C1, C5 to C10, C34 to C11, C35 to C12, C31 to C13, C32 to C14, C6 to C15, C10 to C16, C9 to C17, C7 to C18, C8 to C19, C1 to C2, C2 to C20, C15 to C21, C16 to C22, C17 to C23, C18 to C24, C19 to C25, C27 to C26, C28 to C27, C29 to C28, C22 to C29, C33 to C3, C26 to C30, C23 to C31, C24 to C32, C25 to C33, C11 to C4, C12 to C5, C4 to C6, C3 to C7, C13 to C8, C14 to C9, D2 to D1, D9 to D10, D13 to D11, D14 to D12, D15 to D13, D10 to D14, D11 to D15, D8 to D16, D4 to D17, D6 to D18, D1 to D2, D7 to D20, D16 to D21, D20 to D3, D18 to D4, D19 to D5, D3 to D8, D12 to D9, IC3 to IC1, IC1 to IC2, IC4 to IC3, IC2 to IC4, J3 to J2, J2 to J3, R29 to R1, R5 to R10, R20 to R11, R19 to R12, R18 to R13, R21 to R14, R2 to R15, R3 to R16, R1 to R17, R6 to R18, R8 to R19, R24 to R2, R10 to R20, R7 to R21, R9 to R22, R11 to R23, R15 to R24, R17 to R25, R14 to R26, R16 to R27, R23 to R3, R22 to R4, R25 to R5, R26 to R6, R27 to R7, R28 to R8, R4 to R9, TP2 to TP1, TP1 to TP2
Connections:
- net Net-(JP1-A) renamed /MCU/NRST
- U1 pad 44: unconnected-(U1-XTALHF1/PA0-Pad44) -> /MCU/AUX_UART_TX
- U1 pad 45: unconnected-(U1-XTALHF2/PA1-Pad45) -> /MCU/AUX_UART_RX
- U2 pad 3: unconnected-(U2-PA13-Pad3) -> /MCU/SWDIO
- U2 pad 4: unconnected-(U2-PA14-Pad4) -> /MCU/SWCLK
Routing:
- net /MCU/AUX_UART_TX: track 0.00 -> 57.5 mm, vias 0 -> 1
- net /MCU/AUX_UART_RX: track 0.00 -> 56.6 mm, vias 0 -> 1
- net /MCU/SWDIO: track 0.00 -> 16.2 mm, vias 0 -> 1
- net /MCU/SWCLK: track 0.00 -> 15.2 mm, vias 0 -> 1
- net /MCU/NRST: track 19.7 -> 29.1 mm
- net Net-(D6-K): track 0.00 -> 2.69 mm
- net VCC: track 34.6 -> 36.9 mm, vias 17 -> 18
- net /MCU/RED_LED: track 59.3 -> 61.3 mm
- net GND: track 26.1 -> 27.7 mm
- net Net-(D7-K): track 8.01 -> 7.31 mm
Other:
- board text added: "MowerBoard CAILLIATTE Pierre-Yves V1.0 - 2026 - STAUB 107L16KH"
- board text added: "UART AUX"
- board text added: "UPDI"
- board text removed: "MowerBoard CAILLIATTE Pierre-Yves V1.0 - STAUB 107L16KH"
