File: Hardware/STAUB_BLIZZARD_107L/MowerBoard.kicad_sch (KiCad schematic)
At the start: 11 parts, among them J1 432550083, J2 43045-0227, J3 39-28-1143

Commit message: Travail sur le BOM, changement de quelques empreintes pour aligner sur les disponibilités
Parts:
- J1: footprint Lib:CONN_SDA_43255-00xx_06_MOL -> Custom:CONN_SDA_43255-00xx_06_MOL_NO_MARK
Changed lines of the file:
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@@
 			)
 		)
-		(property "Footprint" "Lib:CONN_SDA_43255-00xx_06_MOL"
+		(property "Footprint" "Custom:CONN_SDA_43255-00xx_06_MOL_NO_MARK"
 			(at 33.02 66.04 0)
 			(hide yes)

Commit message: Ajout du connecteur de programmation du module Lora
Parts:
- renumbered D2 to D1, D1 to D2, D20 to D3, D18 to D4, D19 to D5, J3 to J2, J2 to J3, R29 to R1
Changed lines of the file:
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@@
 		(dnp no)
 		(fields_autoplaced yes)
-		(property "Reference" "D2"
+		(property "Reference" "D1"
 			(at 53.34 24.1299 90)
 			(show_name no)
@@
 			(project "MowerBoard"
 				(path "/bd3c2afb-bb7d-4136-bab9-15428914e155"
-					(reference "D2")
+					(reference "D1")
 					(unit 1)
 				)
@@
 		(dnp no)
 		(fields_autoplaced yes)
-		(property "Reference" "#PWR065"
+		(property "Reference" "#PWR012"
 			(at 106.68 40.64 0)
 			(hide yes)
@@
 			(project "MowerBoard"
 				(path "/bd3c2afb-bb7d-4136-bab9-15428914e155"
-					(reference "#PWR065")
+					(reference "#PWR012")
 					(unit 1)
 				)
@@
 		(dnp no)
 		(fields_autoplaced yes)
-		(property "Reference" "#FLG02"
+		(property "Reference" "#FLG03"
 			(at 86.36 174.625 0)
 			(hide yes)
@@
 			(project "MowerBoard"
 				(path "/bd3c2afb-bb7d-4136-bab9-15428914e155"
-					(reference "#FLG02")
+					(reference "#FLG03")
 					(unit 1)
 				)
@@
 		(dnp no)
 		(fields_autoplaced yes)
-		(property "Reference" "#PWR01"
+		(property "Reference" "#PWR08"
 			(at 86.36 176.53 0)
 			(hide yes)
@@
 			(project "MowerBoard"
 				(path "/bd3c2afb-bb7d-4136-bab9-15428914e155"
-					(reference "#PWR01")
+					(reference "#PWR08")
 					(unit 1)
 				)
@@
 		(in_pos_files yes)
 		(dnp no)
-		(property "Reference" "#PWR030"
+		(property "Reference" "#PWR01"
 			(at 21.59 176.53 0)
 			(hide yes)
@@
 			(project "MowerBoard"
 				(path "/bd3c2afb-bb7d-4136-bab9-15428914e155"
-					(reference "#PWR030")
+					(reference "#PWR01")
 					(unit 1)
 				)
@@
 		(in_pos_files yes)
 		(dnp no)
-		(property "Reference" "#PWR023"
+		(property "Reference" "#PWR03"
 			(at 50.8 41.91 0)
 			(hide yes)
@@
 			(project "MowerBoard"
 				(path "/bd3c2afb-bb7d-4136-bab9-15428914e155"
-					(reference "#PWR023")
+					(reference "#PWR03")
 					(unit 1)
 				)
@@
 		(dnp no)
 		(fields_autoplaced yes)
-		(property "Reference" "#PWR020"
+		(property "Reference" "#PWR04"
 			(at 54.61 87.63 0)
 			(hide yes)
@@
 			(project "MowerBoard"
 				(path "/bd3c2afb-bb7d-4136-bab9-15428914e155"
-					(reference "#PWR020")
+					(reference "#PWR04")
 					(unit 1)
 				)
@@
 		(dnp no)
 		(fields_autoplaced yes)
-		(property "Reference" "D20"
+		(property "Reference" "D3"
 			(at 91.44 62.2299 90)
 			(show_name no)
@@
 			(project "MowerBoard"
 				(path "/bd3c2afb-bb7d-4136-bab9-15428914e155"
-					(reference "D20")
+					(reference "D3")
 					(unit 1)
 				)
@@
 		(dnp no)
 		(fields_autoplaced yes)
-		(property "Reference" "#PWR02"
+		(property "Reference" "#PWR06"
 			(at 67.31 15.24 0)
 			(hide yes)
@@
 			(project "MowerBoard"
 				(path "/bd3c2afb-bb7d-4136-bab9-15428914e155"
-					(reference "#PWR02")
+					(reference "#PWR06")
 					(unit 1)
 				)
@@
 		(dnp no)
 		(fields_autoplaced yes)
-		(property "Reference" "D18"
+		(property "Reference" "D4"
 			(at 118.11 26.6699 90)
 			(show_name no)
@@
 			(project "MowerBoard"
 				(path "/bd3c2afb-bb7d-4136-bab9-15428914e155"
-					(reference "D18")
+					(reference "D4")
 					(unit 1)
 				)
@@
 		(dnp no)
 		(fields_autoplaced yes)
-		(property "Reference" "D19"
+		(property "Reference" "D5"
 			(at 118.11 36.8299 90)
 			(show_name no)
@@
 			(project "MowerBoard"
 				(path "/bd3c2afb-bb7d-4136-bab9-15428914e155"
-					(reference "D19")
+					(reference "D5")
 					(unit 1)
 				)
@@
 		(dnp no)
 		(fields_autoplaced yes)
-		(property "Reference" "#FLG04"
+		(property "Reference" "#FLG02"
 			(at 71.12 61.595 0)
 			(hide yes)
@@
 			(project "MowerBoard"
 				(path "/bd3c2afb-bb7d-4136-bab9-15428914e155"
-					(reference "#FLG04")
+					(reference "#FLG02")
 					(unit 1)
 				)
@@
 		(dnp no)
 		(fields_autoplaced yes)
-		(property "Reference" "#PWR021"
+		(property "Reference" "#PWR05"
 			(at 55.88 130.81 0)
 			(hide yes)
@@
 			(project "MowerBoard"
 				(path "/bd3c2afb-bb7d-4136-bab9-15428914e155"
-					(reference "#PWR021")
+					(reference "#PWR05")
 					(unit 1)
 				)
@@
 		(dnp no)
 		(fields_autoplaced yes)
-		(property "Reference" "D1"
+		(property "Reference" "D2"
 			(at 64.77 31.75 0)
 			(show_name no)
@@
 			(project "MowerBoard"
 				(path "/bd3c2afb-bb7d-4136-bab9-15428914e155"
-					(reference "D1")
+					(reference "D2")
 					(unit 1)
 				)
@@
 		(dnp no)
 		(fields_autoplaced yes)
-		(property "Reference" "#PWR063"
+		(property "Reference" "#PWR09"
 			(at 92.71 45.72 0)
 			(hide yes)
@@
 			(project "MowerBoard"
 				(path "/bd3c2afb-bb7d-4136-bab9-15428914e155"
-					(reference "#PWR063")
+					(reference "#PWR09")
 					(unit 1)
 				)
@@
 		(dnp no)
 		(fields_autoplaced yes)
-		(property "Reference" "J2"
+		(property "Reference" "J3"
 			(at 172.72 96.52 0)
 			(show_name no)
@@
 			(project "MowerBoard"
 				(path "/bd3c2afb-bb7d-4136-bab9-15428914e155"
-					(reference "J2")
+					(reference "J3")
 					(unit 1)
 				)
@@
 		(dnp no)
 		(fields_autoplaced yes)
-		(property "Reference" "#PWR064"
+		(property "Reference" "#PWR011"
 			(at 106.68 30.48 0)
 			(hide yes)
@@
 			(project "MowerBoard"
 				(path "/bd3c2afb-bb7d-4136-bab9-15428914e155"
-					(reference "#PWR064")
+					(reference "#PWR011")
 					(unit 1)
 				)
@@
 		(dnp no)
 		(fields_autoplaced yes)
-		(property "Reference" "#PWR041"
+		(property "Reference" "#PWR013"
 			(at 114.3 152.4 0)
 			(hide yes)
@@
 			(project "MowerBoard"
 				(path "/bd3c2afb-bb7d-4136-bab9-15428914e155"
-					(reference "#PWR041")
+					(reference "#PWR013")
 					(unit 1)
 				)
@@
 		(dnp no)
 		(fields_autoplaced yes)
-		(property "Reference" "#PWR03"
+		(property "Reference" "#PWR02"
 			(at 33.02 55.88 0)
 			(hide yes)
@@
 			(project "MowerBoard"
 				(path "/bd3c2afb-bb7d-4136-bab9-15428914e155"
-					(reference "#PWR03")
+					(reference "#PWR02")
 					(unit 1)
 				)
@@
 		(dnp no)
 		(fields_autoplaced yes)
-		(property "Reference" "R29"
+		(property "Reference" "R1"
 			(at 185.42 95.2499 0)
 			(show_name no)
@@
 			(project "MowerBoard"
 				(path "/bd3c2afb-bb7d-4136-bab9-15428914e155"
-					(reference "R29")
+					(reference "R1")
 					(unit 1)
 				)
@@
 		(dnp no)
 		(fields_autoplaced yes)
-		(property "Reference" "#PWR067"
+		(property "Reference" "#PWR014"
 			(at 182.88 83.82 0)
 			(hide yes)
@@
 			(project "MowerBoard"
 				(path "/bd3c2afb-bb7d-4136-bab9-15428914e155"
-					(reference "#PWR067")
+					(reference "#PWR014")
 					(unit 1)
 				)
@@
 		(dnp no)
 		(fields_autoplaced yes)
-		(property "Reference" "#PWR062"
+		(property "Reference" "#PWR010"
 			(at 109.22 81.28 0)
 			(hide yes)
@@
 			(project "MowerBoard"
 				(path "/bd3c2afb-bb7d-4136-bab9-15428914e155"
-					(reference "#PWR062")
+					(reference "#PWR010")
 					(unit 1)
 				)
@@
 		(dnp no)
 		(fields_autoplaced yes)
-		(property "Reference" "#PWR022"
+		(property "Reference" "#PWR07"
 			(at 71.12 81.28 0)
 			(hide yes)
@@
 			(project "MowerBoard"
 				(path "/bd3c2afb-bb7d-4136-bab9-15428914e155"
-					(reference "#PWR022")
+					(reference "#PWR07")
 					(unit 1)
 				)
@@
 		(dnp no)
 		(fields_autoplaced yes)
-		(property "Reference" "J3"
+		(property "Reference" "J2"
 			(at 143.51 116.84 0)
 			(show_name no)
@@
 			(project "MowerBoard"
 				(path "/bd3c2afb-bb7d-4136-bab9-15428914e155"
-					(reference "J3")
-					(unit 1)
-				)
+					(reference "J2")
+					(unit 1)
+				)
