File: Hardware/STAUB_BLIZZARD_107L/buck.kicad_sch (KiCad schematic)
At the start: 14 parts, among them IC1 TPS62162DSGR, IC4 TPS7B8601QDDARQ1

Commit message: RC2 du PCB, corrigé taille des vias et isolation. Ajout via GND. Reprise des leds de status
Parts:
- TP3: value +5V -> +3.3v
Changed lines of the file:
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@@
 		)
 	)
-	(label "+5v"
+	(label "+3.3v"
 		(at 161.29 115.57 0)
 		(effects
@@
 			)
 		)
-		(property "Value" "+5V"
+		(property "Value" "+3.3v"
 			(at 176.53 113.0299 0)
 			(show_name no)

Commit message: Travail sur le BOM, changement de quelques empreintes pour aligner sur les disponibilités
Parts:
- C10: value 1uF -> 10uF 50V; footprint Capacitor_SMD:C_0805_2012Metric -> Capacitor_SMD:C_1206_3216Metric
- C6: value 10uF -> 10uF 25V
- C7: value 22uF -> 22uF 16V
- C8: value 100uF -> 100uF Polym 10v; symbol Device:C -> Device:C_Polarized
- C9: value 10uF -> 10uF 50V; footprint Capacitor_SMD:C_0805_2012Metric -> Capacitor_SMD:C_1206_3216Metric
- IC4: footprint SamacSys_Parts:SOIC127P600X170-9N -> Custom:SOIC127P600X170-9N_pasta
Other:
- moved on the sheet: C10, R2, R3
Changed lines of the file:
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@@
 	)
 	(junction
-		(at 60.96 54.61)
+		(at 54.61 54.61)
 		(diameter 0)
 		(color 0 0 0 0)
@@
 	)
 	(junction
-		(at 44.45 72.39)
+		(at 38.1 72.39)
 		(diameter 0)
 		(color 0 0 0 0)
@@
 	)
 	(junction
-		(at 44.45 54.61)
+		(at 38.1 54.61)
 		(diameter 0)
 		(color 0 0 0 0)
@@
 	(wire
 		(pts
-			(xy 44.45 54.61) (xy 60.96 54.61)
+			(xy 38.1 54.61) (xy 54.61 54.61)
 		)
 		(stroke
@@
 	(wire
 		(pts
-			(xy 44.45 59.69) (xy 44.45 54.61)
+			(xy 38.1 59.69) (xy 38.1 54.61)
 		)
 		(stroke
@@
 	(wire
 		(pts
-			(xy 44.45 67.31) (xy 44.45 77.47)
+			(xy 38.1 67.31) (xy 38.1 77.47)
 		)
 		(stroke
@@
 	(wire
 		(pts
-			(xy 69.85 72.39) (xy 44.45 72.39)
+			(xy 69.85 72.39) (xy 38.1 72.39)
 		)
 		(stroke
@@
 	(wire
 		(pts
-			(xy 44.45 87.63) (xy 44.45 85.09)
+			(xy 38.1 87.63) (xy 38.1 85.09)
 		)
 		(stroke
@@
 	(wire
 		(pts
-			(xy 60.96 62.23) (xy 60.96 63.5)
+			(xy 54.61 62.23) (xy 54.61 63.5)
 		)
 		(stroke
@@
 	(wire
 		(pts
-			(xy 30.48 54.61) (xy 44.45 54.61)
+			(xy 24.13 54.61) (xy 38.1 54.61)
 		)
 		(stroke
@@
 	(wire
 		(pts
-			(xy 60.96 54.61) (xy 73.66 54.61)
+			(xy 54.61 54.61) (xy 73.66 54.61)
 		)
 		(stroke
@@
 	)
 	(label "+15V_MAX"
-		(at 30.48 54.61 0)
+		(at 24.13 54.61 0)
 		(effects
 			(font
@@
 			)
 		)
-		(property "Value" "10uF"
+		(property "Value" "10uF 50V"
 			(at 125.73 59.6899 0)
 			(show_name no)
@@
 			)
 		)
-		(property "Footprint" "Capacitor_SMD:C_0805_2012Metric"
+		(property "Footprint" "Capacitor_SMD:C_1206_3216Metric"
 			(at 122.8852 62.23 0)
 			(hide yes)
@@
 	(symbol
 		(lib_id "power:GND")
-		(at 44.45 87.63 0)
+		(at 38.1 87.63 0)
 		(unit 1)
 		(body_style 1)
@@
 		(dnp no)
 		(property "Reference" "#PWR026"
-			(at 44.45 93.98 0)
+			(at 38.1 93.98 0)
 			(hide yes)
 			(show_name no)
@@
 		)
 		(property "Value" "GND"
-			(at 48.26 89.154 90)
+			(at 41.91 89.154 90)
 			(show_name no)
 			(do_not_autoplace no)
@@
 		)
 		(property "Footprint" ""
-			(at 44.45 87.63 0)
+			(at 38.1 87.63 0)
 			(hide yes)
 			(show_name no)
@@
 		)
 		(property "Datasheet" ""
-			(at 44.45 87.63 0)
+			(at 38.1 87.63 0)
 			(hide yes)
 			(show_name no)
@@
 		)
 		(property "Description" "Power symbol creates a global label with name \"GND\" , ground"
-			(at 44.45 87.63 0)
+			(at 38.1 87.63 0)
 			(hide yes)
 			(show_name no)
@@
 	(symbol
 		(lib_id "Device:R")
-		(at 44.45 63.5 0)
+		(at 38.1 63.5 0)
 		(unit 1)
 		(body_style 1)
@@
 		(fields_autoplaced yes)
 		(property "Reference" "R2"
-			(at 46.99 62.2299 0)
+			(at 40.64 62.2299 0)
 			(show_name no)
 			(do_not_autoplace no)
@@
 		)
 		(property "Value" "220k"
-			(at 46.99 64.7699 0)
+			(at 40.64 64.7699 0)
 			(show_name no)
 			(do_not_autoplace no)
@@
 		)
 		(property "Footprint" "Resistor_SMD:R_0603_1608Metric"
-			(at 42.672 63.5 90)
+			(at 36.322 63.5 90)
 			(hide yes)
 			(show_name no)
@@
 		)
 		(property "Datasheet" ""
-			(at 44.45 63.5 0)
+			(at 38.1 63.5 0)
 			(hide yes)
 			(show_name no)
@@
 		)
 		(property "Description" "Resistor"
-			(at 44.45 63.5 0)
+			(at 38.1 63.5 0)
 			(hide yes)
 			(show_name no)
@@
 			)
 		)
-		(property "Footprint" "SamacSys_Parts:SOIC127P600X170-9N"
+		(property "Footprint" "Custom:SOIC127P600X170-9N_pasta"
 			(at 100.33 149.53 0)
 			(hide yes)
@@
 	)
 	(symbol
-		(lib_id "Device:C")
+		(lib_id "Device:C_Polarized")
 		(at 161.29 123.19 0)
 		(unit 1)
@@
 		(fields_autoplaced yes)
 		(property "Reference" "C8"
-			(at 165.1 121.9199 0)
+			(at 165.1 121.0309 0)
 			(show_name no)
 			(do_not_autoplace no)
@@
 			)
 		)
-		(property "Value" "100uF"
-			(at 165.1 124.4599 0)
+		(property "Value" "100uF Polym 10v"
+			(at 165.1 123.5709 0)
 			(show_name no)
 			(do_not_autoplace no)
@@
 			)
 		)
-		(property "Description" "Unpolarized capacitor"
+		(property "Description" "Polarized capacitor"
 			(at 161.29 123.19 0)
 			(hide yes)
@@
 	(symbol
 		(lib_id "Device:C")
-		(at 60.96 58.42 0)
+		(at 54.61 58.42 0)
 		(unit 1)
 		(body_style 1)
@@
 		(fields_autoplaced yes)
 		(property "Reference" "C10"
-			(at 64.77 57.1499 0)
+			(at 58.42 57.1499 0)
 			(show_name no)
 			(do_not_autoplace no)
@@
 			)
 		)
-		(property "Value" "1uF"
-			(at 64.77 59.6899 0)
+		(property "Value" "10uF 50V"
+			(at 58.42 59.6899 0)
 			(show_name no)
 			(do_not_autoplace no)
@@
 			)
 		)
-		(property "Footprint" "Capacitor_SMD:C_0805_2012Metric"
-			(at 61.9252 62.23 0)
+		(property "Footprint" "Capacitor_SMD:C_1206_3216Metric"
+			(at 55.5752 62.23 0)
 			(hide yes)
 			(show_name no)
@@
 		)
 		(property "Datasheet" ""
-			(at 60.96 58.42 0)
+			(at 54.61 58.42 0)
 			(hide yes)
 			(show_name no)
@@
 		)
 		(property "Description" "Unpolarized capacitor"
-			(at 60.96 58.42 0)
+			(at 54.61 58.42 0)
 			(hide yes)
 			(show_name no)
@@
 	(symbol
 		(lib_id "Device:R")
-		(at 44.45 81.28 0)
+		(at 38.1 81.28 0)
 		(unit 1)
 		(body_style 1)
@@
 		(fields_autoplaced yes)
 		(property "Reference" "R3"
-			(at 46.99 80.0099 0)
+			(at 40.64 80.0099 0)
 			(show_name no)
 			(do_not_autoplace no)
@@
 		)
 		(property "Value" "10k"
-			(at 46.99 82.5499 0)
+			(at 40.64 82.5499 0)
 			(show_name no)
 			(do_not_autoplace no)
@@
 		)
 		(property "Footprint" "Resistor_SMD:R_0603_1608Metric"
-			(at 42.672 81.28 90)
+			(at 36.322 81.28 90)
 			(hide yes)
 			(show_name no)
@@
 		)
 		(property "Datasheet" ""
-			(at 44.45 81.28 0)
+			(at 38.1 81.28 0)
 			(hide yes)
 			(show_name no)
@@
 		)
 		(property "Description" "Resistor"
-			(at 44.45 81.28 0)
+			(at 38.1 81.28 0)
 			(hide yes)
 			(show_name no)
@@
 	(symbol
 		(lib_id "power:GND")
-		(at 60.96 63.5 0)
+		(at 54.61 63.5 0)
 		(unit 1)
 		(body_style 1)
@@
 		(dnp no)
 		(property "Reference" "#PWR034"
-			(at 60.96 69.85 0)
+			(at 54.61 69.85 0)
 			(hide yes)
 			(show_name no)
@@
 		)
 		(property "Value" "GND"
-			(at 60.96 67.818 0)
+			(at 54.61 67.818 0)
 			(show_name no)
 			(do_not_autoplace no)
@@
 		)
 		(property "Footprint" ""
-			(at 60.96 63.5 0)
+			(at 54.61 63.5 0)
 			(hide yes)
 			(show_name no)
@@
 		)
 		(property "Datasheet" ""
-			(at 60.96 63.5 0)
+			(at 54.61 63.5 0)
 			(hide yes)
 			(show_name no)
@@
 		)
 		(property "Description" "Power symbol creates a global label with name \"GND\" , ground"
-			(at 60.96 63.5 0)
+			(at 54.61 63.5 0)
 			(hide yes)
 			(show_name no)
@@
 			)
 		)
-		(property "Value" "10uF"
+		(property "Value" "10uF 25V"
 			(at 41.91 125.7299 0)
 			(show_name no)
@@
 			)
 		)
-		(property "Value" "22uF"
+		(property "Value" "22uF 16V"
 			(at 149.86 124.4599 0)
 			(show_name no)

Commit message: Ajout du connecteur de programmation du module Lora
Parts:
- renumbered C6 to C15, C10 to C16, C9 to C17, C7 to C18, C8 to C19, IC1 to IC2, IC4 to IC3, R2 to R15, R3 to R16, R1 to R17, TP2 to TP1, TP1 to TP2
