File: Hardware/STAUB_BLIZZARD_107L/io.kicad_sch (KiCad schematic)
At the start: 18 parts, among them IC3 PTPS274C65ASRHAR

Commit message: Travail sur le BOM, changement de quelques empreintes pour aligner sur les disponibilités
Parts:
- added C34: 2.2uF 15V, Capacitor_SMD:C_0603_1608Metric, symbol Device:C_Small
- added C35: 100nF 15V, Capacitor_SMD:C_0402_1005Metric, symbol Device:C_Small
- C31: value 4.7nF -> 4.7nF 50V
- C32: value 100nF -> 100nF 50V
- D8: value D_Schottky_Small -> PMEG60T30ELR-QX
- IC3: footprint SamacSys_Parts:QFN50P600X600X100-41N-D -> Custom:QFN50P600X600X100-41N-D_pasta
- R4, R5: value R_Small -> 390
Connections:
- net GND: now also C34.1, C35.1
- net VCC: now also C34.2, C35.2
Other:
- moved on the sheet: C32

Commit message: Ajout du connecteur de programmation du module Lora
Parts:
- renumbered C34 to C11, C35 to C12, C31 to C13, C32 to C14, D9 to D10, D13 to D11, D14 to D12, D15 to D13, D10 to D14, D11 to D15, D8 to D16, D3 to D8, D12 to D9, IC3 to IC1, R5 to R10, R20 to R11, R19 to R12, R18 to R13, R21 to R14, R4 to R9
