File: Hardware/STAUB_BLIZZARD_107L/mcu.kicad_sch (KiCad schematic)
At the start: 24 parts, among them J4 SMA-J-P-H-ST-TH1, U1 AVR128DB48x-x6LX, U2 317990687

Commit message: Ajout des datasheet, correction des metadata et typo de certain composants.
Parts:
- C11, C13, C33, C4, C5: value 4.7 µF -> 4.7uF
- C12, C14, C3: value 100 nF -> 100nF
- FB1: value FerriteBead_Small -> ILHB0603ER601VHC41
Changed lines of the file:
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@@
 			)
 		)
-		(property "Value" "100 nF"
+		(property "Value" "100nF"
 			(at 67.3036 57.15 90)
 			(show_name no)
@@
 			)
 		)
-		(property "Value" "4.7 µF"
+		(property "Value" "4.7uF"
 			(at 67.056 45.974 90)
 			(show_name no)
@@
 			)
 		)
-		(property "Value" "4.7 µF"
+		(property "Value" "4.7uF"
 			(at 122.936 44.704 90)
 			(show_name no)
@@
 			)
 		)
-		(property "Value" "4.7 µF"
+		(property "Value" "4.7uF"
 			(at 94.996 43.434 90)
 			(show_name no)
@@
 		(fields_autoplaced yes)
 		(property "Reference" "C3"
-			(at 95.2564 64.77 90)
-			(show_name no)
-			(do_not_autoplace no)
-			(effects
-				(font
-					(size 1.27 1.27)
-				)
-			)
-		)
-		(property "Value" "100 nF"
-			(at 95.2564 62.23 90)
+			(at 95.2563 52.07 90)
+			(show_name no)
+			(do_not_autoplace no)
+			(effects
+				(font
+					(size 1.27 1.27)
+				)
+			)
+		)
+		(property "Value" "100nF"
+			(at 95.2563 54.61 90)
 			(show_name no)
 			(do_not_autoplace no)
@@
 		(fields_autoplaced yes)
 		(property "Reference" "C14"
-			(at 123.1964 66.04 90)
-			(show_name no)
-			(do_not_autoplace no)
-			(effects
-				(font
-					(size 1.27 1.27)
-				)
-			)
-		)
-		(property "Value" "100 nF"
-			(at 123.1964 63.5 90)
+			(at 123.1963 53.34 90)
+			(show_name no)
+			(do_not_autoplace no)
+			(effects
+				(font
+					(size 1.27 1.27)
+				)
+			)
+		)
+		(property "Value" "100nF"
+			(at 123.1963 55.88 90)
 			(show_name no)
 			(do_not_autoplace no)
@@
 			)
 		)
-		(property "Value" "4.7 µF"
+		(property "Value" "4.7uF"
 			(at 46.736 61.976 90)
 			(show_name no)
@@
 			)
 		)
-		(property "Value" "4.7 µF"
+		(property "Value" "4.7uF"
 			(at 150.114 80.264 90)
 			(show_name no)
@@
 			)
 		)
-		(property "Value" "FerriteBead_Small"
+		(property "Value" "ILHB0603ER601VHC41"
 			(at 62.992 34.036 0)
 			(show_name no)
@@
 			)
 		)
-		(property "Datasheet" ""
+		(property "Datasheet" "https://www.vishay.com/docs/34690/ilhb-0603.pdf"
 			(at 69.85 40.64 0)
 			(hide yes)

Commit message: Travail sur le BOM, changement de quelques empreintes pour aligner sur les disponibilités
Parts:
- C1: value 1uF -> 1uF 15V
- C11, C13, C33, C4, C5: value 4.7uF -> 4.7uF 15V; footprint Capacitor_SMD:C_0402_1005Metric -> Capacitor_SMD:C_0603_1608Metric
- C12, C14, C3: value 100nF -> 100nF 15V
- C30: value 100pF -> 100pF 15V
- D17: value D_Schottky_Small -> PMEG60T30ELR-QX
- R23: value 1k -> 33k 1/4W
- R24: value 1k -> 100k
- R28: value 22 -> 470
- U1: footprint Package_DFN_QFN:QFN-48-1EP_6x6mm_P0.4mm_EP4.2x4.2mm -> Package_DFN_QFN:VQFN-48-1EP_6x6mm_P0.4mm_EP4.1x4.1mm
Other:
- moved on the sheet: C33
Changed lines of the file:
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@@
 	(wire
 		(pts
-			(xy 30.48 55.88) (xy 40.64 55.88)
+			(xy 30.48 55.88) (xy 44.45 55.88)
 		)
 		(stroke
@@
 	(wire
 		(pts
-			(xy 40.64 55.88) (xy 40.64 59.69)
+			(xy 44.45 55.88) (xy 44.45 59.69)
 		)
 		(stroke
@@
 	(wire
 		(pts
-			(xy 40.64 64.77) (xy 40.64 72.39)
+			(xy 44.45 64.77) (xy 44.45 72.39)
 		)
 		(stroke
@@
 	(wire
 		(pts
-			(xy 30.48 72.39) (xy 40.64 72.39)
+			(xy 30.48 72.39) (xy 44.45 72.39)
 		)
 		(stroke
@@
 			)
 		)
-		(property "Value" "1k"
+		(property "Value" "100k"
 			(at 33.02 41.9099 0)
 			(show_name no)
@@
 		(dnp no)
 		(property "Reference" "C30"
-			(at 20.066 135.89 0)
+			(at 16.51 137.414 0)
 			(show_name no)
 			(do_not_autoplace no)
@@
 			)
 		)
-		(property "Value" "100pF"
-			(at 20.066 138.43 0)
+		(property "Value" "100pF 15V"
+			(at 16.51 139.954 0)
 			(show_name no)
 			(do_not_autoplace no)
@@
 			)
 		)
-		(property "Value" "22"
+		(property "Value" "470"
 			(at 220.98 34.29 90)
 			(show_name no)
@@
 			)
 		)
-		(property "Value" "100nF"
+		(property "Value" "100nF 15V"
 			(at 67.3036 57.15 90)
 			(show_name no)
@@
 			)
 		)
-		(property "Footprint" "Package_DFN_QFN:QFN-48-1EP_6x6mm_P0.4mm_EP4.2x4.2mm"
+		(property "Footprint" "Package_DFN_QFN:VQFN-48-1EP_6x6mm_P0.4mm_EP4.1x4.1mm"
 			(at 86.36 114.3 0)
 			(hide yes)
@@
 			)
 		)
-		(property "Value" "1uF"
+		(property "Value" "1uF 15V"
 			(at 39.37 170.1799 0)
 			(show_name no)
@@
 			)
 		)
-		(property "Value" "4.7uF"
+		(property "Value" "4.7uF 15V"
 			(at 67.056 45.974 90)
 			(show_name no)
@@
 			)
 		)
-		(property "Footprint" "Capacitor_SMD:C_0402_1005Metric"
+		(property "Footprint" "Capacitor_SMD:C_0603_1608Metric"
 			(at 67.31 52.07 0)
 			(hide yes)
@@
 			)
 		)
-		(property "Value" "4.7uF"
+		(property "Value" "4.7uF 15V"
 			(at 122.936 44.704 90)
 			(show_name no)
@@
 			)
 		)
-		(property "Footprint" "Capacitor_SMD:C_0402_1005Metric"
+		(property "Footprint" "Capacitor_SMD:C_0603_1608Metric"
 			(at 123.19 50.8 0)
 			(hide yes)
@@
 			)
 		)
-		(property "Value" "1k"
+		(property "Value" "33k 1/4W"
 			(at 33.02 64.7699 0)
 			(show_name no)
@@
 			)
 		)
-		(property "Value" "4.7uF"
+		(property "Value" "4.7uF 15V"
 			(at 94.996 43.434 90)
 			(show_name no)
@@
 			)
 		)
-		(property "Footprint" "Capacitor_SMD:C_0402_1005Metric"
+		(property "Footprint" "Capacitor_SMD:C_0603_1608Metric"
 			(at 95.25 49.53 0)
 			(hide yes)
@@
 			)
 		)
-		(property "Value" "100nF"
+		(property "Value" "100nF 15V"
 			(at 95.2563 54.61 90)
 			(show_name no)
@@
 			)
 		)
-		(property "Value" "D_Schottky_Small"
+		(property "Value" "PMEG60T30ELR-QX"
 			(at 132.08 143.51 0)
 			(show_name no)
@@
 			)
 		)
-		(property "Value" "100nF"
+		(property "Value" "100nF 15V"
 			(at 123.1963 55.88 90)
 			(show_name no)
@@
 	(symbol
 		(lib_id "Device:C_Small")
-		(at 40.64 62.23 180)
+		(at 44.45 62.23 180)
 		(unit 1)
 		(body_style 1)
@@
 		(dnp no)
 		(property "Reference" "C33"
-			(at 44.196 61.976 90)
+			(at 48.006 61.976 90)
 			(show_name no)
 			(do_not_autoplace no)
@@
 			)
 		)
-		(property "Value" "4.7uF"
-			(at 46.736 61.976 90)
+		(property "Value" "4.7uF 15V"
+			(at 50.546 61.976 90)
 			(show_name no)
 			(do_not_autoplace no)
@@
 			)
 		)
-		(property "Footprint" "Capacitor_SMD:C_0402_1005Metric"
-			(at 40.64 62.23 0)
+		(property "Footprint" "Capacitor_SMD:C_0603_1608Metric"
+			(at 44.45 62.23 0)
 			(hide yes)
 			(show_name no)
@@
 		)
 		(property "Datasheet" ""
-			(at 40.64 62.23 0)
+			(at 44.45 62.23 0)
 			(hide yes)
 			(show_name no)
@@
 		)
 		(property "Description" "Unpolarized capacitor, small symbol"
-			(at 40.64 62.23 0)
+			(at 44.45 62.23 0)
 			(hide yes)
 			(show_name no)
@@
 			)
 		)
-		(property "Value" "4.7uF"
+		(property "Value" "4.7uF 15V"
 			(at 150.114 80.264 90)
 			(show_name no)
@@
 			)
 		)
-		(property "Footprint" "Capacitor_SMD:C_0402_1005Metric"
+		(property "Footprint" "Capacitor_SMD:C_0603_1608Metric"
 			(at 156.21 80.01 0)
 			(hide yes)

Commit message: Ajout du connecteur de programmation du module Lora
Parts:
- removed D17: PMEG60T30ELR-QX, Diode_SMD:Nexperia_CFP3_SOD-123W, symbol Device:D_Schottky_Small
- added D6, D7: BAT54W, Package_TO_SOT_SMD:SOT-323_SC-70, symbol Diode:BAT54W
- added SW1, UART1: (no value), Connector_PinHeader_2.54mm:PinHeader_1x04_P2.54mm_Vertical, symbol Connector_Generic:Conn_01x04
- JP1: now not fitted
- renumbered C30 to C1, C5 to C10, C1 to C2, C33 to C3, C11 to C4, C12 to C5, C4 to C6, C3 to C7, C13 to C8, C14 to C9, R24 to R2, R23 to R3, R22 to R4, R25 to R5, R26 to R6, R27 to R7, R28 to R8
Connections:
- net GND: now also SW1.4 (Pin_4), UART1.4 (Pin_4)
- net VCC: now also D6.1 (A), D7.1 (A)
- net AUX_UART_TX: now reaches U1.44 (XTALHF1/PA0)
- net AUX_UART_TX: now also UART1.3 (Pin_3)
- net AUX_UART_RX: now reaches U1.45 (XTALHF2/PA1)
- net AUX_UART_RX: now also UART1.2 (Pin_2)
- net NRST: now reaches JP1.1 (A), U2.24 (PB13)
- net NRST: now also SW1.3 (Pin_3)
- net SWDIO: now reaches U2.3 (PA13)
- net SWDIO: now also SW1.1 (Pin_1)
- net SWCLK: now reaches U2.4 (PA14)
- net SWCLK: now also SW1.2 (Pin_2)
- net at UPDI1.1 (Pin_1): now also D7.3 (K)
- new net: D6.3 (K), UART1.1 (Pin_1)
- no-connect marks 42 -> 38
