File: Hardware/STAUB_BLIZZARD_107L/relais.kicad_sch (KiCad schematic)
At the start: 6 parts, among them K1 V23086C2001A403, K2 V23086C2001A403

Commit message: Ajout du connecteur de programmation du module Lora
Parts:
- renumbered D4 to D17, D6 to D18, D5 to D19, D7 to D20
Changed lines of the file:
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@@
 		(dnp yes)
 		(fields_autoplaced yes)
-		(property "Reference" "D7"
+		(property "Reference" "D20"
 			(at 170.18 114.2999 90)
 			(show_name no)
@@
 			(project "MowerBoard"
 				(path "/bd3c2afb-bb7d-4136-bab9-15428914e155/c37586b2-d40f-4c7e-8d3e-6ebfc630412f"
-					(reference "D7")
+					(reference "D20")
 					(unit 1)
 				)
@@
 		(dnp yes)
 		(fields_autoplaced yes)
-		(property "Reference" "D6"
+		(property "Reference" "D18"
 			(at 102.87 114.2999 90)
 			(show_name no)
@@
 			(project "MowerBoard"
 				(path "/bd3c2afb-bb7d-4136-bab9-15428914e155/c37586b2-d40f-4c7e-8d3e-6ebfc630412f"
-					(reference "D6")
+					(reference "D18")
 					(unit 1)
 				)
@@
 		(dnp no)
 		(fields_autoplaced yes)
-		(property "Reference" "#PWR032"
+		(property "Reference" "#PWR055"
 			(at 210.82 91.44 0)
 			(hide yes)
@@
 			(project "MowerBoard"
 				(path "/bd3c2afb-bb7d-4136-bab9-15428914e155/c37586b2-d40f-4c7e-8d3e-6ebfc630412f"
-					(reference "#PWR032")
+					(reference "#PWR055")
 					(unit 1)
 				)
@@
 		(dnp no)
 		(fields_autoplaced yes)
-		(property "Reference" "#PWR028"
+		(property "Reference" "#PWR053"
 			(at 63.5 143.51 0)
 			(hide yes)
@@
 			(project "MowerBoard"
 				(path "/bd3c2afb-bb7d-4136-bab9-15428914e155/c37586b2-d40f-4c7e-8d3e-6ebfc630412f"
-					(reference "#PWR028")
+					(reference "#PWR053")
 					(unit 1)
 				)
@@
 		(dnp no)
 		(fields_autoplaced yes)
-		(property "Reference" "#PWR031"
+		(property "Reference" "#PWR052"
 			(at 62.23 92.71 0)
 			(hide yes)
@@
 			(project "MowerBoard"
 				(path "/bd3c2afb-bb7d-4136-bab9-15428914e155/c37586b2-d40f-4c7e-8d3e-6ebfc630412f"
-					(reference "#PWR031")
+					(reference "#PWR052")
 					(unit 1)
 				)
@@
 		(dnp no)
 		(fields_autoplaced yes)
-		(property "Reference" "#PWR029"
+		(property "Reference" "#PWR054"
 			(at 208.28 140.97 0)
 			(hide yes)
@@
 			(project "MowerBoard"
 				(path "/bd3c2afb-bb7d-4136-bab9-15428914e155/c37586b2-d40f-4c7e-8d3e-6ebfc630412f"
-					(reference "#PWR029")
+					(reference "#PWR054")
 					(unit 1)
 				)
@@
 		(dnp yes)
 		(fields_autoplaced yes)
-		(property "Reference" "D4"
+		(property "Reference" "D17"
 			(at 102.87 66.0399 90)
 			(show_name no)
@@
 			(project "MowerBoard"
 				(path "/bd3c2afb-bb7d-4136-bab9-15428914e155/c37586b2-d40f-4c7e-8d3e-6ebfc630412f"
-					(reference "D4")
+					(reference "D17")
 					(unit 1)
 				)
@@
 		(dnp yes)
 		(fields_autoplaced yes)
-		(property "Reference" "D5"
+		(property "Reference" "D19"
 			(at 170.18 66.0399 90)
 			(show_name no)
@@
 			(project "MowerBoard"
 				(path "/bd3c2afb-bb7d-4136-bab9-15428914e155/c37586b2-d40f-4c7e-8d3e-6ebfc630412f"
-					(reference "D5")
+					(reference "D19")
 					(unit 1)
 				)
